File: Arduino Keyboard.sch (EAGLE design)
At the start: 26 parts

Commit message: Version 0.2
Parts:
- renumbered U$10 to SW6, U$11 to SW5, U$12 to SW10, U$13 to SWS4, U$14 to SWS3, U$15 to SW12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
Other:
- note added: "Norbu Borbély III.CI"
