File: Arduino Keyboard.sch (EAGLE design)
At the start: 26 parts, among them SW1 CHERRY-MXSTANDARD, SW10 CHERRY-MXSTANDARD, SW11 CHERRY-MXSTANDARD, SW12 CHERRY-MXSTANDARD, SW13 CHERRY-MXSTANDARD, SW14 CHERRY-MXSTANDARD, SW15 CHERRY-MXSTANDARD, SW16 CHERRY-MXSTANDARD, SW17 CHERRY-MXSTANDARD, SW18 CHERRY-MXSTANDARD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

Commit message: Version 0.4
Parts:
- U$1: device Arduino-clone:NANO -> Arduino-clone_2:NANO
Changed lines of the file:
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@@
 <?xml version="1.0" encoding="utf-8"?>
 <!DOCTYPE eagle SYSTEM "eagle.dtd">
-<eagle version="9.6.2">
+<eagle version="9.6.0">
 <drawing>
 <settings>
@@
 </classes>
 <parts>
-<part name="U$1" library="Arduino-clone" deviceset="NANO" device=""/>
 <part name="SW12" library="cherrymx" deviceset="CHERRY-MX" device="STANDARD"/>
 <part name="SW11" library="cherrymx" deviceset="CHERRY-MX" device="STANDARD"/>
@@
 <part name="SWS5" library="cherrymx" deviceset="CHERRY-MX" device="STANDARD"/>
 <part name="FRAME1" library="frames" library_urn="urn:adsk.eagle:library:229" deviceset="A4L-LOC" device="" value="Norbu Borbély III.CI"/>
+<part name="U$1" library="Arduino-clone_2" deviceset="NANO" device=""/>
 </parts>
 <sheets>
@@
 </plain>
 <instances>
-<instance part="U$1" gate="G$1" x="20.32" y="0" smashed="yes"/>
 <instance part="SW12" gate="G$1" x="91.44" y="43.18" smashed="yes" rot="MR0">
 <attribute name="NAME" x="96.52" y="35.56" size="1.778" layer="95" rot="MR0"/>
@@
 <attribute name="SHEET" x="192.405" y="-38.1" size="2.54" layer="95"/>
 </instance>
+<instance part="U$1" gate="G$1" x="20.32" y="0" smashed="yes"/>
 </instances>
 <busses>
@@
 <net name="N$1" class="0">
 <segment>
-<pinref part="U$1" gate="G$1" pin="D3"/>
 <wire x1="30.48" y1="-7.62" x2="78.74" y2="-7.62" width="0.1524" layer="91"/>
 <wire x1="78.74" y1="-7.62" x2="78.74" y2="0" width="0.1524" layer="91"/>
@@
 <wire x1="104.14" y1="0" x2="101.6" y2="0" width="0.1524" layer="91"/>
 <junction x="104.14" y="-7.62"/>
+<pinref part="U$1" gate="G$1" pin="D3"/>
 </segment>
 </net>
 <net name="N$2" class="0">
 <segment>
-<pinref part="U$1" gate="G$1" pin="D4"/>
 <wire x1="30.48" y1="-5.08" x2="55.88" y2="-5.08" width="0.1524" layer="91"/>
 <wire x1="55.88" y1="-5.08" x2="55.88" y2="12.7" width="0.1524" layer="91"/>
@@
 <wire x1="78.74" y1="20.32" x2="76.2" y2="20.32" width="0.1524" layer="91"/>
 <junction x="78.74" y="12.7"/>
+<pinref part="U$1" gate="G$1" pin="D4"/>
 </segment>
 </net>
 <net name="N$3" class="0">
 <segment>
-<pinref part="U$1" gate="G$1" pin="D5"/>
 <wire x1="30.48" y1="-2.54" x2="53.34" y2="-2.54" width="0.1524" layer="91"/>
 <wire x1="53.34" y1="-2.54" x2="53.34" y2="33.02" width="0.1524" layer="91"/>
@@
 <wire x1="78.74" y1="40.64" x2="76.2" y2="40.64" width="0.1524" layer="91"/>
 <junction x="78.74" y="33.02"/>
+<pinref part="U$1" gate="G$1" pin="D5"/>
 </segment>
 </net>
 <net name="N$4" class="0">
 <segment>
-<pinref part="U$1" gate="G$1" pin="D6"/>
 <wire x1="30.48" y1="0" x2="50.8" y2="0" width="0.1524" layer="91"/>
 <wire x1="50.8" y1="0" x2="50.8" y2="53.34" width="0.1524" layer="91"/>
@@
 <wire x1="78.74" y1="60.96" x2="76.2" y2="60.96" width="0.1524" layer="91"/>
 <junction x="78.74" y="53.34"/>
+<pinref part="U$1" gate="G$1" pin="D6"/>
 </segment>
 </net>
 <net name="N$5" class="0">
 <segment>
-<pinref part="U$1" gate="G$1" pin="D7"/>
 <wire x1="30.48" y1="2.54" x2="48.26" y2="2.54" width="0.1524" layer="91"/>
 <wire x1="48.26" y1="2.54" x2="48.26" y2="73.66" width="0.1524" layer="91"/>
@@
 <wire x1="78.74" y1="81.28" x2="76.2" y2="81.28" width="0.1524" layer="91"/>
 <junction x="78.74" y="73.66"/>
+<pinref part="U$1" gate="G$1" pin="D7"/>
 </segment>
 </net>
 <net name="N$6" class="0">
 <segment>
-<pinref part="U$1" gate="G$1" pin="D8"/>
 <wire x1="30.48" y1="5.08" x2="45.72" y2="5.08" width="0.1524" layer="91"/>
 <wire x1="45.72" y1="5.08" x2="45.72" y2="93.98" width="0.1524" layer="91"/>
@@
 <wire x1="76.2" y1="66.04" x2="81.28" y2="66.04" width="0.1524" layer="91"/>
 <junction x="81.28" y="66.04"/>
+<pinref part="U$1" gate="G$1" pin="D8"/>
 </segment>
 </net>
 <net name="N$7" class="0">
 <segment>
-<pinref part="U$1" gate="G$1" pin="D9"/>
 <wire x1="30.48" y1="7.62" x2="43.18" y2="7.62" width="0.1524" layer="91"/>
 <wire x1="43.18" y1="7.62" x2="43.18" y2="96.52" width="0.1524" layer="91"/>
@@
 <wire x1="101.6" y1="86.36" x2="106.68" y2="86.36" width="0.1524" layer="91"/>
 <junction x="106.68" y="86.36"/>
+<pinref part="U$1" gate="G$1" pin="D9"/>
 </segment>
 </net>
 <net name="N$8" class="0">
 <segment>
-<pinref part="U$1" gate="G$1" pin="D10"/>
 <wire x1="30.48" y1="10.16" x2="40.64" y2="10.16" width="0.1524" layer="91"/>
 <wire x1="40.64" y1="10.16" x2="40.64" y2="99.06" width="0.1524" layer="91"/>
@@
 <wire x1="127" y1="86.36" x2="132.08" y2="86.36" width="0.1524" layer="91"/>
 <junction x="132.08" y="86.36"/>
+<pinref part="U$1" gate="G$1" pin="D10"/>
 </segment>
 </net>
 <net name="N$9" class="0">
 <segment>
-<pinref part="U$1" gate="G$1" pin="D11"/>
 <wire x1="30.48" y1="12.7" x2="38.1" y2="12.7" width="0.1524" layer="91"/>
 <wire x1="38.1" y1="12.7" x2="38.1" y2="101.6" width="0.1524" layer="91"/>
@@
 <wire x1="152.4" y1="86.36" x2="157.48" y2="86.36" width="0.1524" layer="91"/>
 <junction x="157.48" y="86.36"/>
+<pinref part="U$1" gate="G$1" pin="D11"/>
 </segment>
 </net>
 <net name="N$10" class="0">
 <segment>
-<pinref part="U$1" gate="G$1" pin="D12"/>
 <wire x1="30.48" y1="15.24" x2="35.56" y2="15.24" width="0.1524" layer="91"/>
 <wire x1="35.56" y1="15.24" x2="35.56" y2="104.14" width="0.1524" layer="91"/>
@@
 <wire x1="177.8" y1="86.36" x2="182.88" y2="86.36" width="0.1524" layer="91"/>
 <junction x="182.88" y="86.36"/>
-</segment>
-</net>
+<pinref part="U$1" gate="G$1" pin="D12"/>
+</segment>
+</net>
